File: KiCad Files/Pump_Control_Board.kicad_pcb (KiCad board)
At the start: 2 copper layers, 64 x 56 mm, 70 parts, among them J1 OLED, J2 Conn_01x06, J3 USB_C_Receptacle_USB2.0, J4 Jack, M1 Stepper_Motor_bipolar, Q1 SSM3J328R, SW1 SW_USER, SW2 SW_RESET, U1 ESDALD05, U2 SN74LV1T34DCK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

Commit message: Named ICP Header
Parts:
- J2: value Conn_01x06 -> ICP Header
Changed lines of the file:
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@@
         (effects (font (size 1 1) (thickness 0.15)))
     )
-    (fp_text value "Conn_01x06" (at 0 15.03) (layer "F.Fab")
+    (fp_text value "ICP Header" (at 0 15.03) (layer "F.Fab")
         (effects (font (size 1 1) (thickness 0.15)))
     )
